File: pcb/comfybox.kicad_sch (KiCad schematic)
At the start: 20 parts, among them K1 SW_CHOC, K2 SW_CHOC, K3 SW_CHOC, K4 SW_CHOC, P1 SW_CHOC, P2 SW_CHOC, P3 SW_CHOC, P4 SW_CHOC

Commit message: layout adjustments and MX compatibility
Parts:
- DOWN1, K1, K2, K3, K4, LEFT1, P1, P2, P3, P4, RIGHT1, UP1, UP2: footprint Switch:Kailh_PG1350_Gateron_KS27_KS33 -> Switch:Kailh_PG1350_Gateron_KS33_MX
Changed lines of the file:
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@@
     (property "Reference" "LEFT1" (id 0) (at 120.65 64.77 0))
     (property "Value" "SW_CHOC" (id 1) (at 120.65 67.31 0))
-    (property "Footprint" "Switch:Kailh_PG1350_Gateron_KS27_KS33" (id 2) (at 120.65 67.31 0)
+    (property "Footprint" "Switch:Kailh_PG1350_Gateron_KS33_MX" (id 2) (at 120.65 67.31 0)
       (effects (font (size 1.27 1.27)) hide)
     )
@@
     (property "Reference" "K4" (id 0) (at 181.61 111.76 0))
     (property "Value" "SW_CHOC" (id 1) (at 181.61 114.3 0))
-    (property "Footprint" "Switch:Kailh_PG1350_Gateron_KS27_KS33" (id 2) (at 181.61 114.3 0)
+    (property "Footprint" "Switch:Kailh_PG1350_Gateron_KS33_MX" (id 2) (at 181.61 114.3 0)
       (effects (font (size 1.27 1.27)) hide)
     )
@@
     (property "Reference" "K2" (id 0) (at 140.97 111.76 0))
     (property "Value" "SW_CHOC" (id 1) (at 140.97 114.3 0))
-    (property "Footprint" "Switch:Kailh_PG1350_Gateron_KS27_KS33" (id 2) (at 140.97 114.3 0)
+    (property "Footprint" "Switch:Kailh_PG1350_Gateron_KS33_MX" (id 2) (at 140.97 114.3 0)
       (effects (font (size 1.27 1.27)) hide)
     )
@@
     (property "Reference" "UP2" (id 0) (at 201.93 64.77 0))
     (property "Value" "SW_CHOC" (id 1) (at 201.93 67.31 0))
-    (property "Footprint" "Switch:Kailh_PG1350_Gateron_KS27_KS33" (id 2) (at 201.93 67.31 0)
+    (property "Footprint" "Switch:Kailh_PG1350_Gateron_KS33_MX" (id 2) (at 201.93 67.31 0)
       (effects (font (size 1.27 1.27)) hide)
     )
@@
     (property "Reference" "P1" (id 0) (at 120.65 90.17 0))
     (property "Value" "SW_CHOC" (id 1) (at 120.65 92.71 0))
-    (property "Footprint" "Switch:Kailh_PG1350_Gateron_KS27_KS33" (id 2) (at 120.65 92.71 0)
+    (property "Footprint" "Switch:Kailh_PG1350_Gateron_KS33_MX" (id 2) (at 120.65 92.71 0)
       (effects (font (size 1.27 1.27)) hide)
     )
@@
     (property "Reference" "K3" (id 0) (at 161.29 111.76 0))
     (property "Value" "SW_CHOC" (id 1) (at 161.29 114.3 0))
-    (property "Footprint" "Switch:Kailh_PG1350_Gateron_KS27_KS33" (id 2) (at 161.29 114.3 0)
+    (property "Footprint" "Switch:Kailh_PG1350_Gateron_KS33_MX" (id 2) (at 161.29 114.3 0)
       (effects (font (size 1.27 1.27)) hide)
     )
@@
     (property "Reference" "P4" (id 0) (at 181.61 90.17 0))
     (property "Value" "SW_CHOC" (id 1) (at 181.61 92.71 0))
-    (property "Footprint" "Switch:Kailh_PG1350_Gateron_KS27_KS33" (id 2) (at 181.61 92.71 0)
+    (property "Footprint" "Switch:Kailh_PG1350_Gateron_KS33_MX" (id 2) (at 181.61 92.71 0)
       (effects (font (size 1.27 1.27)) hide)
     )
@@
     (property "Reference" "P3" (id 0) (at 161.29 90.17 0))
     (property "Value" "SW_CHOC" (id 1) (at 161.29 92.71 0))
-    (property "Footprint" "Switch:Kailh_PG1350_Gateron_KS27_KS33" (id 2) (at 161.29 92.71 0)
+    (property "Footprint" "Switch:Kailh_PG1350_Gateron_KS33_MX" (id 2) (at 161.29 92.71 0)
       (effects (font (size 1.27 1.27)) hide)
     )
@@
     (property "Reference" "DOWN1" (id 0) (at 140.97 64.77 0))
     (property "Value" "SW_CHOC" (id 1) (at 140.97 67.31 0))
-    (property "Footprint" "Switch:Kailh_PG1350_Gateron_KS27_KS33" (id 2) (at 140.97 67.31 0)
+    (property "Footprint" "Switch:Kailh_PG1350_Gateron_KS33_MX" (id 2) (at 140.97 67.31 0)
       (effects (font (size 1.27 1.27)) hide)
     )
@@
   (symbol (lib_id "power:GND") (at 54.61 130.81 0) (unit 1)
     (in_bom yes) (on_board yes) (fields_autoplaced)
-    (property "Reference" "#PWR?" (id 0) (at 54.61 137.16 0)
+    (property "Reference" "#PWR0101" (id 0) (at 54.61 137.16 0)
       (effects (font (size 1.27 1.27)) hide)
     )
@@
     (property "Reference" "K1" (id 0) (at 120.65 111.76 0))
     (property "Value" "SW_CHOC" (id 1) (at 120.65 114.3 0))
-    (property "Footprint" "Switch:Kailh_PG1350_Gateron_KS27_KS33" (id 2) (at 120.65 114.3 0)
+    (property "Footprint" "Switch:Kailh_PG1350_Gateron_KS33_MX" (id 2) (at 120.65 114.3 0)
       (effects (font (size 1.27 1.27)) hide)
     )
@@
     (property "Reference" "P2" (id 0) (at 140.97 90.17 0))
     (property "Value" "SW_CHOC" (id 1) (at 140.97 92.71 0))
-    (property "Footprint" "Switch:Kailh_PG1350_Gateron_KS27_KS33" (id 2) (at 140.97 92.71 0)
+    (property "Footprint" "Switch:Kailh_PG1350_Gateron_KS33_MX" (id 2) (at 140.97 92.71 0)
       (effects (font (size 1.27 1.27)) hide)
     )
@@
     (property "Reference" "UP1" (id 0) (at 181.61 64.77 0))
     (property "Value" "SW_CHOC" (id 1) (at 181.61 67.31 0))
-    (property "Footprint" "Switch:Kailh_PG1350_Gateron_KS27_KS33" (id 2) (at 181.61 67.31 0)
+    (property "Footprint" "Switch:Kailh_PG1350_Gateron_KS33_MX" (id 2) (at 181.61 67.31 0)
       (effects (font (size 1.27 1.27)) hide)
     )
@@
     (property "Reference" "RIGHT1" (id 0) (at 161.29 64.77 0))
     (property "Value" "SW_CHOC" (id 1) (at 161.29 67.31 0))
-    (property "Footprint" "Switch:Kailh_PG1350_Gateron_KS27_KS33" (id 2) (at 161.29 67.31 0)
+    (property "Footprint" "Switch:Kailh_PG1350_Gateron_KS33_MX" (id 2) (at 161.29 67.31 0)
       (effects (font (size 1.27 1.27)) hide)
     )
@@
     )
     (path "/8ebb64d1-1b87-45bc-8a21-f86410e35966"
-      (reference "#PWR?") (unit 1) (value "GND") (footprint "")
+      (reference "#PWR0101") (unit 1) (value "GND") (footprint "")
     )
     (path "/7d452c23-f08c-4cf7-8335-8028ad6af654"
-      (reference "DOWN1") (unit 1) (value "SW_CHOC") (footprint "Switch:Kailh_PG1350_Gateron_KS27_KS33")
+      (reference "DOWN1") (unit 1) (value "SW_CHOC") (footprint "Switch:Kailh_PG1350_Gateron_KS33_MX")
     )
     (path "/988573a5-ea42-45d3-9cd1-0c53b1863f2e"
-      (reference "K1") (unit 1) (value "SW_CHOC") (footprint "Switch:Kailh_PG1350_Gateron_KS27_KS33")
+      (reference "K1") (unit 1) (value "SW_CHOC") (footprint "Switch:Kailh_PG1350_Gateron_KS33_MX")
     )
     (path "/15ec41f1-698a-4727-beef-17758bb95787"
-      (reference "K2") (unit 1) (value "SW_CHOC") (footprint "Switch:Kailh_PG1350_Gateron_KS27_KS33")
+      (reference "K2") (unit 1) (value "SW_CHOC") (footprint "Switch:Kailh_PG1350_Gateron_KS33_MX")
     )
     (path "/727e679b-e0d3-41f0-96a9-aff13fe9cbb4"
-      (reference "K3") (unit 1) (value "SW_CHOC") (footprint "Switch:Kailh_PG1350_Gateron_KS27_KS33")
+      (reference "K3") (unit 1) (value "SW_CHOC") (footprint "Switch:Kailh_PG1350_Gateron_KS33_MX")
     )
     (path "/0c9cf060-b141-4ba5-9990-940b1fe0ad3f"
-      (reference "K4") (unit 1) (value "SW_CHOC") (footprint "Switch:Kailh_PG1350_Gateron_KS27_KS33")
+      (reference "K4") (unit 1) (value "SW_CHOC") (footprint "Switch:Kailh_PG1350_Gateron_KS33_MX")
     )
     (path "/07666484-4233-43b6-8b39-89daeb01304c"
-      (reference "LEFT1") (unit 1) (value "SW_CHOC") (footprint "Switch:Kailh_PG1350_Gateron_KS27_KS33")
+      (reference "LEFT1") (unit 1) (value "SW_CHOC") (footprint "Switch:Kailh_PG1350_Gateron_KS33_MX")
     )
     (path "/85c97a58-edb1-46c2-952a-8c8e5519c14c"
@@
     )
     (path "/6da0731c-10c2-4953-ae34-8d25ba0f01a3"
-      (reference "P1") (unit 1) (value "SW_CHOC") (footprint "Switch:Kailh_PG1350_Gateron_KS27_KS33")
+      (reference "P1") (unit 1) (value "SW_CHOC") (footprint "Switch:Kailh_PG1350_Gateron_KS33_MX")
     )
     (path "/cd5f6696-504a-44a7-903f-e0a955615676"
-      (reference "P2") (unit 1) (value "SW_CHOC") (footprint "Switch:Kailh_PG1350_Gateron_KS27_KS33")
+      (reference "P2") (unit 1) (value "SW_CHOC") (footprint "Switch:Kailh_PG1350_Gateron_KS33_MX")
     )
     (path "/7c7f925c-6407-4bcd-88a8-6de65100b0dc"
-      (reference "P3") (unit 1) (value "SW_CHOC") (footprint "Switch:Kailh_PG1350_Gateron_KS27_KS33")
+      (reference "P3") (unit 1) (value "SW_CHOC") (footprint "Switch:Kailh_PG1350_Gateron_KS33_MX")
     )
     (path "/7936b223-b7bd-4515-a0fe-d144ab49b05f"
-      (reference "P4") (unit 1) (value "SW_CHOC") (footprint "Switch:Kailh_PG1350_Gateron_KS27_KS33")
+      (reference "P4") (unit 1) (value "SW_CHOC") (footprint "Switch:Kailh_PG1350_Gateron_KS33_MX")
     )
     (path "/e76e705b-1acd-49f8-917b-6c87709d07ea"
-      (reference "RIGHT1") (unit 1) (value "SW_CHOC") (footprint "Switch:Kailh_PG1350_Gateron_KS27_KS33")
+      (reference "RIGHT1") (unit 1) (value "SW_CHOC") (footprint "Switch:Kailh_PG1350_Gateron_KS33_MX")
     )
     (path "/1c88fcf1-197e-4669-a023-1e1afa0350b1"
@@
     )
     (path "/ce8a3f3c-1400-4998-82a3-592704bb4069"
-      (reference "UP1") (unit 1) (value "SW_CHOC") (footprint "Switch:Kailh_PG1350_Gateron_KS27_KS33")
+      (reference "UP1") (unit 1) (value "SW_CHOC") (footprint "Switch:Kailh_PG1350_Gateron_KS33_MX")
     )
     (path "/2bf912dd-be99-4601-b086-b60d1966be39"
-      (reference "UP2") (unit 1) (value "SW_CHOC") (footprint "Switch:Kailh_PG1350_Gateron_KS27_KS33")
-    )
-  )
+      (reference "UP2") (unit 1) (value "SW_CHOC") (footprint "Switch:Kailh_PG1350_Gateron_KS33_MX")
+    )
+  )

Commit message: reversible rp2040
Parts:
- DOWN1, K1, K2, K3, K4, LEFT1, P1, P2, P3, P4, RIGHT1, UP1, UP2: footprint Switch:Kailh_PG1350_Gateron_KS33_MX -> Switch:Kailh_PG1350_Gateron_KS33_MX_reversible
- RPZ1: footprint RP2040-Zero:RP2040-Zero -> RP2040-Zero:RP2040-Zero_reversible
Changed lines of the file:
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@@
       (effects (font (size 1.27 1.27)))
     )
-    (property "Footprint" "Switch:Kailh_PG1350_Gateron_KS33_MX" (at 120.65 67.31 0)
+    (property "Footprint" "Switch:Kailh_PG1350_Gateron_KS33_MX_reversible" (at 120.65 67.31 0)
       (effects (font (size 1.27 1.27)) hide)
     )
@@
       (effects (font (size 1.27 1.27)))
     )
-    (property "Footprint" "Switch:Kailh_PG1350_Gateron_KS33_MX" (at 181.61 114.3 0)
+    (property "Footprint" "Switch:Kailh_PG1350_Gateron_KS33_MX_reversible" (at 181.61 114.3 0)
       (effects (font (size 1.27 1.27)) hide)
     )
@@
       (effects (font (size 1.27 1.27)))
     )
-    (property "Footprint" "Switch:Kailh_PG1350_Gateron_KS33_MX" (at 140.97 114.3 0)
+    (property "Footprint" "Switch:Kailh_PG1350_Gateron_KS33_MX_reversible" (at 140.97 114.3 0)
       (effects (font (size 1.27 1.27)) hide)
     )
@@
       (effects (font (size 1.27 1.27)) (justify left))
     )
-    (property "Footprint" "RP2040-Zero:RP2040-Zero" (at 62.23 67.31 0)
+    (property "Footprint" "RP2040-Zero:RP2040-Zero_reversible" (at 62.23 67.31 0)
       (effects (font (size 1.27 1.27)) hide)
     )
@@
       (effects (font (size 1.27 1.27)))
     )
-    (property "Footprint" "Switch:Kailh_PG1350_Gateron_KS33_MX" (at 201.93 67.31 0)
+    (property "Footprint" "Switch:Kailh_PG1350_Gateron_KS33_MX_reversible" (at 201.93 67.31 0)
       (effects (font (size 1.27 1.27)) hide)
     )
@@
       (effects (font (size 1.27 1.27)))
     )
-    (property "Footprint" "Switch:Kailh_PG1350_Gateron_KS33_MX" (at 120.65 92.71 0)
+    (property "Footprint" "Switch:Kailh_PG1350_Gateron_KS33_MX_reversible" (at 120.65 92.71 0)
       (effects (font (size 1.27 1.27)) hide)
     )
@@
       (effects (font (size 1.27 1.27)))
     )
-    (property "Footprint" "Switch:Kailh_PG1350_Gateron_KS33_MX" (at 161.29 114.3 0)
+    (property "Footprint" "Switch:Kailh_PG1350_Gateron_KS33_MX_reversible" (at 161.29 114.3 0)
       (effects (font (size 1.27 1.27)) hide)
     )
@@
       (effects (font (size 1.27 1.27)))
     )
-    (property "Footprint" "Switch:Kailh_PG1350_Gateron_KS33_MX" (at 181.61 92.71 0)
+    (property "Footprint" "Switch:Kailh_PG1350_Gateron_KS33_MX_reversible" (at 181.61 92.71 0)
       (effects (font (size 1.27 1.27)) hide)
     )
@@
       (effects (font (size 1.27 1.27)))
     )
-    (property "Footprint" "Switch:Kailh_PG1350_Gateron_KS33_MX" (at 161.29 92.71 0)
+    (property "Footprint" "Switch:Kailh_PG1350_Gateron_KS33_MX_reversible" (at 161.29 92.71 0)
       (effects (font (size 1.27 1.27)) hide)
     )
@@
       (effects (font (size 1.27 1.27)))
     )
-    (property "Footprint" "Switch:Kailh_PG1350_Gateron_KS33_MX" (at 140.97 67.31 0)
+    (property "Footprint" "Switch:Kailh_PG1350_Gateron_KS33_MX_reversible" (at 140.97 67.31 0)
       (effects (font (size 1.27 1.27)) hide)
     )
@@
       (effects (font (size 1.27 1.27)))
     )
-    (property "Footprint" "Switch:Kailh_PG1350_Gateron_KS33_MX" (at 120.65 114.3 0)
+    (property "Footprint" "Switch:Kailh_PG1350_Gateron_KS33_MX_reversible" (at 120.65 114.3 0)
       (effects (font (size 1.27 1.27)) hide)
     )
@@
       (effects (font (size 1.27 1.27)))
     )
-    (property "Footprint" "Switch:Kailh_PG1350_Gateron_KS33_MX" (at 140.97 92.71 0)
+    (property "Footprint" "Switch:Kailh_PG1350_Gateron_KS33_MX_reversible" (at 140.97 92.71 0)
       (effects (font (size 1.27 1.27)) hide)
     )
@@
       (effects (font (size 1.27 1.27)))
     )
-    (property "Footprint" "Switch:Kailh_PG1350_Gateron_KS33_MX" (at 181.61 67.31 0)
+    (property "Footprint" "Switch:Kailh_PG1350_Gateron_KS33_MX_reversible" (at 181.61 67.31 0)
       (effects (font (size 1.27 1.27)) hide)
     )
@@
       (effects (font (size 1.27 1.27)))
     )
-    (property "Footprint" "Switch:Kailh_PG1350_Gateron_KS33_MX" (at 161.29 67.31 0)
-      (effects (font (size 1.27 1.27)) hide)
-    )
+    (property "Footprint" "Switch:Kailh_PG1350_Gateron_KS33_MX_reversible" (at 161.29 67.31 0)
+      (effects (font (size 1.27 1.27)) hide)
+    )
